File: FOC_Driver.kicad_pcb (KiCad board)
At the start: 2 copper layers, 24 parts, among them J1 Conn_01x06_Pin, J2 Conn_01x03, J3 Conn_02x17_Odd_Even, SW1 SW_MEC_5E, U1 AMS1117-3.3, U2 STM32H503RBTx, Y1 Crystal

Commit message: Wip
Parts:
- removed D2: LED, LED_SMD:LED_0805_2012Metric_Pad1.15x1.40mm_HandSolder
- added C13: 100n, Capacitor_SMD:C_0805_2012Metric_Pad1.18x1.45mm_HandSolder, F.Cu at (60.0, 120.4)
- added C14: 100n, Capacitor_SMD:C_0805_2012Metric_Pad1.18x1.45mm_HandSolder, F.Cu at (60.0, 123.4)
- added C15: 100n, Capacitor_SMD:C_0805_2012Metric_Pad1.18x1.45mm_HandSolder, F.Cu at (97.0, 82.1)
- added C16: 100n, Capacitor_SMD:C_0805_2012Metric_Pad1.18x1.45mm_HandSolder, F.Cu at (97.0, 85.1)
- added J4: DE9_Socket, Connector_Dsub:DSUB-9_Pins_EdgeMount_P2.77mm, F.Cu at (46.0, 98.2)
- added J5: RJ45, Connector_RJ:RJ45_Amphenol_54602-x08_Horizontal, F.Cu at (42.1, 59.7)
- added J6: RJ45, Connector_RJ:RJ45_Amphenol_54602-x08_Horizontal, F.Cu at (42.4, 40.8)
- added R10: R, Resistor_SMD:R_0805_2012Metric_Pad1.20x1.40mm_HandSolder, F.Cu at (99.2, 113.3)
- added R11: R, Resistor_SMD:R_0805_2012Metric_Pad1.20x1.40mm_HandSolder, F.Cu at (99.2, 116.2)
- added R12: 120, Resistor_SMD:R_0805_2012Metric, F.Cu at (92.7, 98.5)
- added R13: 120, Resistor_SMD:R_0805_2012Metric, F.Cu at (92.7, 101.5)
- added R14: 120, Resistor_SMD:R_0805_2012Metric, F.Cu at (92.7, 104.5)
- added R15: 1k, Resistor_SMD:R_0805_2012Metric, F.Cu at (92.7, 107.4)
- added R16: 1k, Resistor_SMD:R_0805_2012Metric, F.Cu at (92.7, 110.3)
- added R17: 10k, Resistor_SMD:R_0805_2012Metric, F.Cu at (92.7, 113.3)
- added R18: 50, Resistor_SMD:R_0805_2012Metric, F.Cu at (92.7, 116.2)
- added R19: 120, Resistor_SMD:R_0805_2012Metric, F.Cu at (85.0, 130.0)
- added R4: R, Resistor_SMD:R_0805_2012Metric_Pad1.20x1.40mm_HandSolder, F.Cu at (99.2, 98.5)
- added R5: R, Resistor_SMD:R_0805_2012Metric_Pad1.20x1.40mm_HandSolder, F.Cu at (99.2, 101.5)
- added R6: R, Resistor_SMD:R_0805_2012Metric_Pad1.20x1.40mm_HandSolder, F.Cu at (99.2, 104.5)
- added R7: R, Resistor_SMD:R_0805_2012Metric_Pad1.20x1.40mm_HandSolder, F.Cu at (99.2, 107.4)
- added R9: R, Resistor_SMD:R_0805_2012Metric_Pad1.20x1.40mm_HandSolder, F.Cu at (99.2, 110.3)
- added U3: AM26LS32ACDR, AM26L32ACDR:SOIC127P600X175-16N, F.Cu at (74.8, 99.0)
- added U4: AP2151AW-7, AP2151:SOT95P285X140-5N, F.Cu at (74.5, 89.0)
- added U5: GD25D10CT, Package_SO:JEITA_SOIC-8_3.9x4.9mm_P1.27mm, F.Cu at (111.3, 85.1)
- C12: value 10u -> 100n
- R8: value R -> 120; footprint Resistor_SMD:R_0805_2012Metric_Pad1.20x1.40mm_HandSolder -> Resistor_SMD:R_0805_2012Metric
- U1: value AMS1117-3.3 -> ST485E; footprint Package_TO_SOT_SMD:SOT-223-3_TabPin2 -> Package_SO:SOIC-8_3.9x4.9mm_P1.27mm
- moved R8 75.9 mm to (88.0, 130.0), turned to -90 degrees
- moved C12 65.9 mm to (109.6, 89.8)
- moved J3 12.2 mm to (139.3, 41.7)
- moved U1 11.5 mm to (56.3, 64.0)
- moved C11 9.06 mm to (59.0, 58.0)
Connections:
- C11 pad 1: VCC_External -> GNDS
- C11 pad 2: GNDD -> Net-(U1-VCC)
- R8 pad 1: +3.3V -> Net-(U1-RO)
- R8 pad 2: Net-(D2-A) -> Net-(U1-~{RE})
- U1 pad 1: GNDD -> Net-(U1-RO)
- U1 pad 2: +3.3V -> Net-(U1-~{RE})
- U1 pad 3: VCC_External -> Net-(U1-DE)

Commit message: wip
Parts:
- removed R11: R, Resistor_SMD:R_0805_2012Metric_Pad1.20x1.40mm_HandSolder
- removed R19: 120, Resistor_SMD:R_0805_2012Metric
- removed U2: STM32H503RBTx, Package_QFP:LQFP-64_10x10mm_P0.5mm
- added C15: 100n, Capacitor_SMD:C_0805_2012Metric_Pad1.18x1.45mm_HandSolder, F.Cu at (201.0, 130.0)
- added C16: 100n, Capacitor_SMD:C_0805_2012Metric_Pad1.18x1.45mm_HandSolder, F.Cu at (201.0, 127.0)
- added IC1: 131M61, 131M61:SOIC127P1030X265-16N, F.Cu at (174.0, 92.0)
- added U6: STM32H523RCTx, Package_QFP:LQFP-64_10x10mm_P0.5mm, F.Cu at (143.0, 89.0)
- J3: footprint Connector_IDC:IDC-Header_2x17_P2.54mm_Horizontal -> Connector_IDC:IDC-Header_2x17_P2.54mm_Vertical
- J4: footprint Connector_Dsub:DSUB-9_Pins_EdgeMount_P2.77mm -> Connector_Dsub:DSUB-9_Socket_Vertical_P2.77x2.84mm_MountingHoles
- J5, J6: footprint Connector_RJ:RJ45_Amphenol_54602-x08_Horizontal -> Connector_RJ:RJ45_OST_PJ012-8P8CX_Vertical
- R10, R4, R5, R6, R7, R9: value R -> 50
- moved C11 169.0 mm to (211.0, 132.0), turned to -90 degrees
- moved J6 159.9 mm to (191.4, 98.6), turned to 90 degrees
- moved J5 150.9 mm to (191.7, 79.7), turned to 90 degrees
- moved C6 138.4 mm to (189.0, 129.0), turned to 180 degrees
- moved C7 135.4 mm to (189.0, 126.0), turned to 180 degrees
- moved C8 132.6 mm to (189.0, 123.0), turned to 180 degrees
- moved J2 125.1 mm to (153.0, 134.5), turned to 180 degrees
- moved C1 122.6 mm to (142.8, 142.8), turned to 180 degrees
- moved C14 119.2 mm to (166.0, 69.0), turned to 90 degrees
- moved U1 118.7 mm to (174.5, 73.9)
- moved C2 117.6 mm to (142.8, 139.8), turned to 180 degrees
- moved C3 112.6 mm to (142.8, 136.8), turned to 180 degrees
- moved C13 109.0 mm to (156.0, 69.0), turned to -90 degrees
- moved R8 108.6 mm to (181.0, 73.9)
- moved C4 107.8 mm to (142.8, 133.8), turned to 180 degrees
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Connections:
- C13 pad 2: +3.3V -> /Encoder/5V_Encoder
- J3 pad 1: /Connectors/EM_STOP -> /Connectors/Disable_Drive
- J3 pad 31: /Connectors/Encoder_A -> unconnected-(J3-Pin_31-Pad31)
- J3 pad 33: /Connectors/Encoder_B -> unconnected-(J3-Pin_33-Pad33)
- J3 pad 34: /Connectors/Encoder_C -> unconnected-(J3-Pin_34-Pad34)
- R10 pad 1: unconnected-(R10-Pad1) -> /MCU/CH1N
- R10 pad 2: unconnected-(R10-Pad2) -> /Connectors/PWM_AL
- R16 pad 1: +3.3V -> /Encoder/5V_Encoder
- R17 pad 2: +5V -> +3.3V
- R4 pad 1: unconnected-(R4-Pad1) -> /MCU/CH3
- R4 pad 2: unconnected-(R4-Pad2) -> /Connectors/PWM_CH
- R5 pad 1: unconnected-(R5-Pad1) -> /MCU/CH2
- R5 pad 2: unconnected-(R5-Pad2) -> /Connectors/PWM_BH
- R6 pad 1: unconnected-(R6-Pad1) -> /MCU/CH1
- R6 pad 2: unconnected-(R6-Pad2) -> /Connectors/PWM_AH
- R7 pad 1: unconnected-(R7-Pad1) -> /Connectors/PWM_CL
- R7 pad 2: unconnected-(R7-Pad2) -> /MCU/CH3N
- R8 pad 1: Net-(U1-RO) -> Net-(U1-B)
- R8 pad 2: Net-(U1-~{RE}) -> Net-(U1-A)
- R9 pad 1: unconnected-(R9-Pad1) -> /MCU/CH2N
- R9 pad 2: unconnected-(R9-Pad2) -> /Connectors/PWM_BL
- U1 pad 1: Net-(U1-RO) -> Net-(IC1-VIC)
- U1 pad 2: Net-(U1-~{RE}) -> Net-(IC1-VOA)
- U1 pad 3: Net-(U1-DE) -> Net-(IC1-VOA)
- U3 pad 16: +3.3V -> /Encoder/5V_Encoder

Commit message: wip
Parts:
- added C17: 1u, Capacitor_SMD:C_0805_2012Metric, F.Cu at (89.5, 126.6)
- added C18: 1u, Capacitor_SMD:C_0805_2012Metric, F.Cu at (89.5, 129.6)
- added C19: 1u, Capacitor_SMD:C_0805_2012Metric, F.Cu at (89.5, 132.7)
- added C20: 1u, Capacitor_SMD:C_0805_2012Metric, F.Cu at (89.5, 135.7)
- added Q1: BSS138, Package_TO_SOT_SMD:SOT-23, F.Cu at (222.1, 68.0)
- added Q2: BSS138, Package_TO_SOT_SMD:SOT-23, F.Cu at (218.0, 68.0)
- added Q3: BSS138, Package_TO_SOT_SMD:SOT-23, F.Cu at (214.0, 68.0)
- added R11: 10k, Resistor_SMD:R_0805_2012Metric, F.Cu at (227.0, 68.0)
- added R19: 10k, Resistor_SMD:R_0805_2012Metric, F.Cu at (230.0, 64.0)
- added R20: 10k, Resistor_SMD:R_0805_2012Metric, F.Cu at (229.1, 72.0)
- added R21: 10k, Resistor_SMD:R_0805_2012Metric, F.Cu at (229.0, 75.0)
- added R22: 10k, Resistor_SMD:R_0805_2012Metric, F.Cu at (229.1, 78.0)
- added R23: 10k, Resistor_SMD:R_0805_2012Metric, F.Cu at (229.1, 80.9)
- added U2: AZ1117-3.3, Package_TO_SOT_SMD:SOT-223-3_TabPin2, F.Cu at (180.0, 123.1)
- added U7: AZ1117-5.0, Package_TO_SOT_SMD:SOT-223-3_TabPin2, F.Cu at (180.0, 133.1)
- C1: value C -> 100n
- moved J2 7.87 mm to (158.0, 128.5), turned to 0 degrees
- moved J3 3.00 mm to (118.0, 98.3)
- moved U5 1.00 mm to (133.0, 71.0), turned to 0 degrees
Connections:
- net /RS485/RS485_DE renamed /MCU/RS485_DE
- net /RS485/RS485_Rx renamed /MCU/RS485_Rx
- net /RS485/RS485_Tx renamed /MCU/RS485_Tx
- C11 pad 2: Net-(U1-VCC) -> VCC_ISO
- C16 pad 1: unconnected-(C16-Pad1) -> VCC_ISO
- IC1 pad 10: Net-(IC1-EN2) -> VCC_ISO
- IC1 pad 15: GNDS -> GND_ISO
- IC1 pad 16: Net-(IC1-EN2) -> VCC_ISO
- IC1 pad 9: GNDS -> GND_ISO
- J5 pad 1: unconnected-(J5-Pad1) -> VCC_ISO
- J5 pad 2: unconnected-(J5-Pad2) -> VCC_ISO
- J5 pad 3: unconnected-(J5-Pad3) -> VCC_ISO
- J5 pad 4: unconnected-(J5-Pad4) -> Net-(U1-B)
- J5 pad 5: unconnected-(J5-Pad5) -> Net-(U1-A)
- J5 pad 6: unconnected-(J5-Pad6) -> GND_ISO
- J5 pad 7: unconnected-(J5-Pad7) -> GND_ISO
- J5 pad 8: unconnected-(J5-Pad8) -> GND_ISO
- J6 pad 1: unconnected-(J6-Pad1) -> VCC_ISO
- J6 pad 2: unconnected-(J6-Pad2) -> VCC_ISO
- J6 pad 3: unconnected-(J6-Pad3) -> VCC_ISO
- J6 pad 4: unconnected-(J6-Pad4) -> Net-(U1-B)
- J6 pad 5: unconnected-(J6-Pad5) -> Net-(U1-A)
- J6 pad 6: unconnected-(J6-Pad6) -> GND_ISO
- J6 pad 7: unconnected-(J6-Pad7) -> GND_ISO
- J6 pad 8: unconnected-(J6-Pad8) -> GND_ISO
- U1 pad 5: GNDS -> GND_ISO
- U1 pad 8: Net-(U1-VCC) -> VCC_ISO
- U3 pad 13: /Encoder/Encoder_0 -> Net-(Q3-D)
- U3 pad 3: /Encoder/Encoder_A -> Net-(Q1-D)
- U3 pad 5: /Encoder/Encoder_B -> Net-(Q2-D)
- U6 pad 12: unconnected-(U6-VSSA-Pad12) -> GNDD
- U6 pad 18: Net-(U6-VSS-Pad18) -> GNDD
- U6 pad 31: Net-(U6-VSS-Pad18) -> GNDD
- U6 pad 47: Net-(U6-VSS-Pad18) -> GNDD
- U6 pad 63: Net-(U6-VSS-Pad18) -> GNDD
Other:
- board outline added: 154 x 119 mm

Commit message: 90% schematic first layout
Parts:
- removed the C15 at (100.3, 84.4)
- removed the C16 at (100.3, 81.4)
- removed Y1: Crystal, Crystal:Crystal_SMD_HC49-SD
- added C21: 100n, Capacitor_SMD:C_0805_2012Metric_Pad1.18x1.45mm_HandSolder, F.Cu at (143.2, 64.2)
- added C22: 100n, Capacitor_SMD:C_0805_2012Metric_Pad1.18x1.45mm_HandSolder, F.Cu at (143.2, 60.2)
- added C23: 1u, Capacitor_SMD:C_0805_2012Metric_Pad1.18x1.45mm_HandSolder, F.Cu at (208.5, 140.2)
- added C24: 1u, Capacitor_SMD:C_0805_2012Metric_Pad1.18x1.45mm_HandSolder, F.Cu at (208.8, 147.8)
- added D1: BZT52B-c12x, Diode_SMD:D_SOD-123F, F.Cu at (132.7, 151.2)
- added J7: Screw_Terminal_01x16, TerminalBlock:TerminalBlock_Xinya_XY308-2.54-16P_1x16_P2.54mm_Horizontal, F.Cu at (185.8, 90.5)
- added L1: 8.2u, Inductor_SMD:L_6.3x6.3_H3, F.Cu at (138.9, 161.5)
- added Q4: MMBT2222A, Package_TO_SOT_SMD:SOT-23, F.Cu at (230.1, 133.3)
- added Q5: BSS138, Package_TO_SOT_SMD:SOT-23, F.Cu at (229.8, 148.1)
- added R24: 100k, Resistor_SMD:R_0805_2012Metric, F.Cu at (226.2, 133.1)
- added R25: 10k, Resistor_SMD:R_0805_2012Metric, F.Cu at (224.2, 133.1)
- added R26: 1k, Resistor_SMD:R_0805_2012Metric, F.Cu at (224.4, 143.3)
- added R27: 100k, Resistor_SMD:R_0805_2012Metric, F.Cu at (226.4, 143.3)
- added R28: 1k, Resistor_SMD:R_0805_2012Metric, F.Cu at (224.4, 148.1)
- added R29: 100k, Resistor_SMD:R_0805_2012Metric, F.Cu at (226.4, 148.1)
- added R30: 10k, Resistor_SMD:R_0805_2012Metric, F.Cu at (132.8, 64.2)
- added R31: 50, Resistor_SMD:R_0805_2012Metric_Pad1.20x1.40mm_HandSolder, F.Cu at (145.0, 78.0)
- added R32: 50, Resistor_SMD:R_0805_2012Metric_Pad1.20x1.40mm_HandSolder, F.Cu at (143.0, 78.0)
- added R33: 50, Resistor_SMD:R_0805_2012Metric_Pad1.20x1.40mm_HandSolder, F.Cu at (141.0, 78.0)
- added R34: 50, Resistor_SMD:R_0805_2012Metric_Pad1.20x1.40mm_HandSolder, F.Cu at (139.0, 78.0)
- added SW3: SW_Push, Button_Switch_THT:SW_PUSH_6mm_H5mm, F.Cu at (212.5, 138.0)
- added SW4: SW_Push, Button_Switch_THT:SW_PUSH_6mm_H5mm, F.Cu at (212.5, 145.5)
- added TP1: TestPoint, TestPoint:TestPoint_Pad_D1.0mm, F.Cu at (212.8, 107.2)
- added U8: 4504, Package_SO:SOIC-16_3.9x9.9mm_P1.27mm, F.Cu at (150.5, 62.2)
- added U9: TSR1-2450E, Converter_DCDC:Converter_DCDC_TRACO_TSR1-xxxxE_THT, F.Cu at (132.2, 168.2)
- C17, C18: value 1u -> 4.7u
- C19: value 1u -> 100n
- C20: value 1u -> 10u
- J4: footprint Connector_Dsub:DSUB-9_Socket_Vertical_P2.77x2.84mm_MountingHoles -> Connector_Dsub:DSUB-9_Pins_Horizontal_P2.77x2.84mm_EdgePinOffset4.94mm_Housed_MountingHolesOffset4.94mm
- J6: footprint Connector_RJ:RJ45_OST_PJ012-8P8CX_Vertical -> Connector_RJ:RJ45_Amphenol_54602-x08_Horizontal
- Q1: value BSS138 -> AOD413A; footprint Package_TO_SOT_SMD:SOT-23 -> AOD413A:AOD413A
- R1: value R -> 10k
- R15, R16: value 1k -> 10k
- R19: value 10k -> 100k; footprint Resistor_SMD:R_0805_2012Metric -> Resistor_SMD:R_0805_2012Metric_Pad1.20x1.40mm_HandSolder
- R20, R21, R22: value 10k -> 100k
- R23: value 10k -> 1k
- SW1: value SW_MEC_5E -> SW_Push; footprint Button_Switch_SMD:SW_MEC_5GSH9 -> Button_Switch_THT:SW_PUSH_6mm_H5mm
- U7: value AZ1117-5.0 -> CSTNE8M00G550000R0; footprint Package_TO_SOT_SMD:SOT-223-3_TabPin2 -> CSTNE8:CSTNE16M0V530000R0
- moved R19 134.5 mm to (127.4, 151.0), turned to -90 degrees
- moved Q1 114.9 mm to (143.4, 151.8), turned to -90 degrees
- moved J2 105.0 mm to (56.0, 103.5)
- moved J1 87.1 mm to (67.5, 50.9), turned to 180 degrees
- moved SW1 81.5 mm to (212.5, 130.5), turned to 0 degrees
- moved Q3 77.1 mm to (229.8, 143.4)
- moved R11 77.0 mm to (150.8, 57.0)
- moved R21 76.3 mm to (206.0, 147.8), turned to -90 degrees
- moved U2 75.2 mm to (128.5, 178.0), turned to 180 degrees
- moved R18 72.3 mm to (163.2, 74.7), turned to -90 degrees
- moved Q2 71.8 mm to (229.8, 138.8)
- moved R20 71.8 mm to (206.5, 140.2), turned to 90 degrees
- moved C7 70.7 mm to (137.0, 78.0), turned to 90 degrees
- moved C15 67.9 mm to (138.7, 103.0), turned to 90 degrees
- moved J6 67.8 mm to (127.1, 120.2), turned to 0 degrees
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Connections:
- net /External_Memory/MISO renamed /MCU/MISO
- net /External_Memory/MOSI renamed /MCU/MOSI
- net /External_Memory/SCLK renamed /MCU/SCLK
- net /External_Memory/nCS renamed /MCU/nCS
- C17 pad 2: +15V -> Net-(U9-Vin)
- C18 pad 2: +5V -> Net-(D1-K)
- Q1 pad 1: +3.3V -> Net-(D1-A)
- Q1 pad 2: /Encoder/Encoder_A -> +24V
- Q1 pad 3: Net-(Q1-D) -> Net-(D1-K)
- Q2 pad 1: +3.3V -> Net-(Q2-G)
- Q2 pad 2: /Encoder/Encoder_B -> GNDD
- Q2 pad 3: Net-(Q2-D) -> ERROR_LED-
- Q3 pad 1: +3.3V -> Net-(Q3-G)
- Q3 pad 2: /Encoder/Encoder_0 -> GNDD
- Q3 pad 3: Net-(Q3-D) -> RUN_LED-
- R11 pad 1: +5V -> /Encoder/5V_Encoder
- R11 pad 2: Net-(Q1-D) -> Net-(U8-Select)
- R19 pad 1: /Encoder/Encoder_A -> Net-(D1-A)
- R19 pad 2: +3.3V -> GNDD
- R20 pad 1: +5V -> +3.3V
- R20 pad 2: Net-(Q2-D) -> RUN/STOP
- R21 pad 1: /Encoder/Encoder_B -> +3.3V
- R21 pad 2: +3.3V -> Error_Fixed
- R22 pad 1: +5V -> Net-(Q2-G)
- R22 pad 2: Net-(Q3-D) -> GNDD
- R23 pad 1: /Encoder/Encoder_0 -> /MCU/ERROR_LED
- R23 pad 2: +3.3V -> Net-(Q2-G)
- SW1 pad 2: GNDD -> /MCU/NRST
- U3 pad 13: Net-(Q3-D) -> Net-(U3-4Y)
- U3 pad 3: Net-(Q1-D) -> Net-(U3-1Y)
- U3 pad 5: Net-(Q2-D) -> Net-(U3-2Y)
- U5 pad 3: /External_Memory/nWP -> Net-(U5-~{WP})
- U7 pad 1: GNDD -> /MCU/RCC_In
- U7 pad 2: +5V -> GNDD
- U7 pad 3: +15V -> /MCU/RCC_Out
Routing:
- net Net-(U3-4Y): track 0.00 -> 11.2 mm
- net /MCU/RCC_Out: track 0.00 -> 4.49 mm
- net /MCU/RCC_In: track 0.00 -> 4.45 mm
- net /Encoder//B: track 0.00 -> 3.34 mm
- net Net-(U3-~{G}): track 0.00 -> 3.33 mm
- net Net-(U3-G): track 0.00 -> 3.25 mm
- net /Encoder//0: track 0.00 -> 3.24 mm
- net /Encoder//A: track 0.00 -> 3.14 mm
- net /Encoder/0: track 0.00 -> 3.14 mm
- net /Encoder/B: track 0.00 -> 3.11 mm
- net /Encoder/A: track 0.00 -> 3.08 mm
Other:
- board size 154 x 119 mm -> 86 x 84.2 mm
