File: Power.kicad_sch (KiCad schematic)
At the start: 6 parts, among them U2 AZ1117-3.3, U7 AZ1117-5.0

Commit message: 90% schematic first layout
Parts:
- removed U7: AZ1117-5.0, Package_TO_SOT_SMD:SOT-223-3_TabPin2, symbol Regulator_Linear:AZ1117-5.0
- added D1: BZT52B-c12x, Diode_SMD:D_SOD-123F, symbol Diode:BZT52Bxx
- added L1: 8.2u, Inductor_SMD:L_6.3x6.3_H3, symbol Device:L
- added Q1: AOD413A, AOD413A, symbol AOD413A:AOD413A
- added R19: 100k, Resistor_SMD:R_0805_2012Metric_Pad1.20x1.40mm_HandSolder, symbol Device:R
- added U9: TSR1-2450E, Converter_DCDC:Converter_DCDC_TRACO_TSR1-xxxxE_THT, symbol Regulator_Switching:TSR1-2450E
- C17, C18: value 1u -> 4.7u
- C19: value 1u -> 100n
- C20: value 1u -> 10u
Connections:
- net +5V: now also U9.3 (Vout); no longer C18.2
- net GNDD: now also R19.2, U9.2 (GND)
- net +15V: no longer names the net of C17.2
- net +15V: now also L1.2, U9.1 (Vin)
- new net: D1.2 (A), Q1.1 (G), R19.1
- new net: C18.2, D1.1 (K), L1.1, Q1.3 (S)
- new net +24V: Q1.2 (D)
Other:
- note removed: "Reverse Polarity Diode? ESD? Header?"
- moved on the sheet: C19, C20, U2

Commit message: Addition of testpoints
Parts:
- added Q9: ZXMP4A16G, Package_TO_SOT_SMD:SOT-223-3_TabPin2, symbol Transistor_FET:ZXMP4A16G
Connections:
- net +24V: now also Q9.2 (D); no longer Q1.2 (D)
- net at D1.2 (A), R19.1: now also Q9.1 (G); no longer Q1.1 (G)
- net at C18.2, D1.1 (K), L1.1: now also Q9.3 (S); no longer Q1.3 (S)
Other:
- moved on the sheet: Q1
Changed lines of the file:
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@@
 	(wire
 		(pts
-			(xy 151.13 38.1) (xy 151.13 39.37)
-		)
-		(stroke
-			(width 0)
-			(type default)
-		)
-	)
-	(wire
-		(pts
-			(xy 31.75 39.37) (xy 34.29 39.37)
+			(xy 151.13 36.83) (xy 151.13 39.37)
+		)
+		(stroke
+			(width 0)
+			(type default)
+		)
+	)
+	(wire
+		(pts
+			(xy 31.75 39.37) (xy 39.37 39.37)
 		)
 		(stroke
@@
 	(symbol
 		(lib_id "AOD413A:AOD413A")
-		(at 44.45 46.99 90)
+		(at 71.12 33.02 90)
 		(unit 1)
 		(exclude_from_sim no)
@@
 		(fields_autoplaced yes)
 		(property "Reference" "Q1"
-			(at 41.91 31.75 90)
+			(at 68.58 17.78 90)
 			(effects
 				(font
@@
 		)
 		(property "Value" "AOD413A"
-			(at 41.91 34.29 90)
+			(at 68.58 20.32 90)
 			(effects
 				(font
@@
 		)
 		(property "Footprint" "AOD413A"
-			(at 143.18 35.56 0)
+			(at 169.85 21.59 0)
 			(effects
 				(font
@@
 		)
 		(property "Datasheet" "https://www.aosmd.com/res/datasheets/AOD413A.pdf"
-			(at 243.18 35.56 0)
+			(at 269.85 21.59 0)
 			(effects
 				(font
@@
 		)
 		(property "Description" "Trans MOSFET P-CH 40V 12A 3-Pin(2+Tab) DPAK"
-			(at 44.45 46.99 0)
+			(at 71.12 33.02 0)
 			(effects
 				(font
@@
 		)
 		(property "Height" "2.6"
-			(at 443.18 35.56 0)
+			(at 469.85 21.59 0)
 			(effects
 				(font
@@
 		)
 		(property "TME Electronic Components Part Number" ""
-			(at 543.18 35.56 0)
+			(at 569.85 21.59 0)
 			(effects
 				(font
@@
 		)
 		(property "TME Electronic Components Price/Stock" ""
-			(at 643.18 35.56 0)
+			(at 669.85 21.59 0)
 			(effects
 				(font
@@
 		)
 		(property "Manufacturer_Name" "Alpha & Omega Semiconductors"
-			(at 743.18 35.56 0)
+			(at 769.85 21.59 0)
 			(effects
 				(font
@@
 		)
 		(property "Manufacturer_Part_Number" "AOD413A"
-			(at 843.18 35.56 0)
+			(at 869.85 21.59 0)
 			(effects
 				(font
@@
 		)
 		(instances
-			(project ""
+			(project "FOC_Driver"
 				(path "/d122ff09-cd02-4f53-acb5-49b9ee3003a4/9e9712b1-28dc-4627-8025-e4634456cce2"
 					(reference "Q1")
@@
 	(symbol
 		(lib_id "power:+3.3V")
-		(at 151.13 38.1 0)
+		(at 151.13 36.83 0)
 		(unit 1)
 		(exclude_from_sim no)
@@
 		(fields_autoplaced yes)
 		(property "Reference" "#PWR063"
-			(at 151.13 41.91 0)
+			(at 151.13 40.64 0)
 			(effects
 				(font
@@
 		)
 		(property "Value" "+3.3V"
-			(at 151.13 33.02 0)
+			(at 151.13 31.75 0)
 			(effects
 				(font
@@
 		)
 		(property "Footprint" ""
-			(at 151.13 38.1 0)
+			(at 151.13 36.83 0)
 			(effects
 				(font
@@
 		)
 		(property "Datasheet" ""
-			(at 151.13 38.1 0)
+			(at 151.13 36.83 0)
 			(effects
 				(font
@@
 		)
 		(property "Description" "Power symbol creates a global label with name \"+3.3V\""
-			(at 151.13 38.1 0)
+			(at 151.13 36.83 0)
 			(effects
 				(font
@@
 					(unit 1)
 				)
+			)
+		)
+	)
+	(symbol
+		(lib_id "Transistor_FET:ZXMP4A16G")
+		(at 44.45 41.91 90)
+		(unit 1)
+		(exclude_from_sim no)
+		(in_bom yes)
+		(on_board yes)
+		(dnp no)
+		(fields_autoplaced yes)
+		(property "Reference" "Q9"
+			(at 44.45 33.02 90)
+			(effects
+				(font
+					(size 1.27 1.27)
+				)
+			)
+		)
+		(property "Value" "ZXMP4A16G"
+			(at 44.45 35.56 90)
+			(effects
+				(font
+					(size 1.27 1.27)
+				)
+			)
+		)
+		(property "Footprint" "Package_TO_SOT_SMD:SOT-223-3_TabPin2"
+			(at 46.355 36.83 0)
+			(effects
+				(font
+					(size 1.27 1.27)
+					(italic yes)
+				)
+				(justify left)
+				(hide yes)
+			)
+		)
+		(property "Datasheet" "https://www.diodes.com/assets/Datasheets/ZXMP4A16G.pdf"
+			(at 48.26 36.83 0)
+			(effects
+				(font
+					(size 1.27 1.27)
+				)
+				(justify left)
+				(hide yes)
+			)
+		)
+		(property "Description" "-6.4A Id, -40V Vds, P-Channel MOSFET, SOT-223"
+			(at 44.45 41.91 0)
+			(effects
+				(font
+					(size 1.27 1.27)
+				)
+				(hide yes)
+			)
+		)
+		(pin "3"
+		)
+		(pin "2"
+		)
+		(pin "1"
+		)
+		(instances
+			(project "FOC_Driver"
+				(path "/d122ff09-cd02-4f53-acb5-49b9ee3003a4/9e9712b1-28dc-4627-8025-e4634456cce2"
+					(reference "Q9")
+					(unit 1)
+				)
